File: maxim-optimizer/maxim-optimizer.kicad_pcb (KiCad board)
At the start: 2 copper layers, 80 x 45 mm, 73 parts, among them U201 MAX20801, U301 MAX20801, U401 MAX20801

Commit message: as ordered
Parts:
- added Item101: Item, t14_team14-logo:team14-logo-icon-0.47, F.Cu at (70.2, 97.8)
- added Item102: Item, t14_team14-logo:team14-logo-schrift-0.47, F.Cu at (71.7, 97.6)
Routing:
- net /Out+: vias 0 -> 22
- added copper zone on B.Cu, net /Out+
Other:
- board text added: "Karl Zeilhofer"
- board text added: "Maxim Optimizer v20.0.0"
