File: maxim-optimizer/optimizer.sch (KiCad schematic (older format))
At the start: 20 parts, among them U201 MAX20801

Commit message: as ordered
Changed lines of the file:
@@
 AR Path="/5F69D945/5F65C68C" Ref="U301"  Part="1"
 AR Path="/5F69D9BA/5F65C68C" Ref="U401"  Part="1"
-F 0 "U301" H 5100 4000 50  0000 L CNN
+F 0 "U401" H 5100 4000 50  0000 L CNN
 F 1 "MAX20801" H 5900 3300 50  0000 L CNN
 F 2 "maxim-optimizer:MAX20801" H 6050 2700 50  0001 C CNN
@@
 AR Path="/5F69D945/5F65CF26" Ref="C312"  Part="1"
 AR Path="/5F69D9BA/5F65CF26" Ref="C412"  Part="1"
-F 0 "C312" H 4815 4238 40  0000 L CNN
+F 0 "C412" H 4815 4238 40  0000 L CNN
 F 1 "1u/6V3" H 4815 4162 40  0000 L CNN
 F 2 "t14_standardSMD:C1608m" V 4850 4200 30  0001 C CNN
@@
 AR Path="/5F69D945/5F65D08A" Ref="C313"  Part="1"
 AR Path="/5F69D9BA/5F65D08A" Ref="C413"  Part="1"
-F 0 "C313" H 6315 3438 40  0000 L CNN
+F 0 "C413" H 6315 3438 40  0000 L CNN
 F 1 "220n/6V3" H 6315 3362 40  0000 L CNN
 F 2 "t14_standardSMD:C1608m" V 6350 3400 30  0001 C CNN
@@
 AR Path="/5F69D945/5F65FA9A" Ref="L301"  Part="1"
 AR Path="/5F69D9BA/5F65FA9A" Ref="L401"  Part="1"
-F 0 "L301" V 6790 3750 50  0000 C CNN
+F 0 "L401" V 6790 3750 50  0000 C CNN
 F 1 "WE-7443739650068" V 6700 3650 50  0000 C CNN
 F 2 "maxim-optimizer:WE-LHMI_1365" H 6600 3750 50  0001 C CNN
@@
 AR Path="/5F69D945/5F66CEBD" Ref="C308"  Part="1"
 AR Path="/5F69D9BA/5F66CEBD" Ref="C408"  Part="1"
-F 0 "C308" V 3750 4350 40  0000 L CNN
+F 0 "C408" V 3750 4350 40  0000 L CNN
 F 1 "100n/25V" V 3850 4300 40  0000 L CNN
 F 2 "t14_standardSMD:C1608m" V 3950 4200 30  0001 C CNN
@@
 AR Path="/5F69D945/5F673CE1" Ref="C301"  Part="1"
 AR Path="/5F69D9BA/5F673CE1" Ref="C401"  Part="1"
-F 0 "C301" V 2250 4350 40  0000 L CNN
+F 0 "C401" V 2250 4350 40  0000 L CNN
 F 1 "10u/25V" V 2350 4300 40  0000 L CNN
 F 2 "t14_standardSMD:C2012m" V 2450 4200 30  0001 C CNN
@@
 AR Path="/5F69D945/5F696E50" Ref="C302"  Part="1"
 AR Path="/5F69D9BA/5F696E50" Ref="C402"  Part="1"
-F 0 "C302" V 2450 4350 40  0000 L CNN
+F 0 "C402" V 2450 4350 40  0000 L CNN
 F 1 "10u/25V" V 2550 4300 40  0000 L CNN
 F 2 "t14_standardSMD:C2012m" V 2650 4200 30  0001 C CNN
@@
 AR Path="/5F69D945/5F697068" Ref="C303"  Part="1"
 AR Path="/5F69D9BA/5F697068" Ref="C403"  Part="1"
-F 0 "C303" V 2650 4350 40  0000 L CNN
+F 0 "C403" V 2650 4350 40  0000 L CNN
 F 1 "10u/25V" V 2750 4300 40  0000 L CNN
 F 2 "t14_standardSMD:C2012m" V 2850 4200 30  0001 C CNN
@@
 AR Path="/5F69D945/5F697239" Ref="C304"  Part="1"
 AR Path="/5F69D9BA/5F697239" Ref="C404"  Part="1"
-F 0 "C304" V 2850 4350 40  0000 L CNN
+F 0 "C404" V 2850 4350 40  0000 L CNN
 F 1 "10u/25V" V 2950 4300 40  0000 L CNN
 F 2 "t14_standardSMD:C2012m" V 3050 4200 30  0001 C CNN
@@
 AR Path="/5F69D945/5F69758E" Ref="C305"  Part="1"
 AR Path="/5F69D9BA/5F69758E" Ref="C405"  Part="1"
-F 0 "C305" V 3050 4350 40  0000 L CNN
+F 0 "C405" V 3050 4350 40  0000 L CNN
 F 1 "10u/25V" V 3150 4300 40  0000 L CNN
 F 2 "t14_standardSMD:C2012m" V 3250 4200 30  0001 C CNN
@@
 AR Path="/5F69D945/5F69782B" Ref="C306"  Part="1"
 AR Path="/5F69D9BA/5F69782B" Ref="C406"  Part="1"
-F 0 "C306" V 3250 4350 40  0000 L CNN
+F 0 "C406" V 3250 4350 40  0000 L CNN
 F 1 "10u/25V" V 3350 4300 40  0000 L CNN
 F 2 "t14_standardSMD:C2012m" V 3450 4200 30  0001 C CNN
@@
 AR Path="/5F69D945/5F6979D1" Ref="C307"  Part="1"
 AR Path="/5F69D9BA/5F6979D1" Ref="C407"  Part="1"
-F 0 "C307" V 3450 4350 40  0000 L CNN
+F 0 "C407" V 3450 4350 40  0000 L CNN
 F 1 "10u/25V" V 3550 4300 40  0000 L CNN
 F 2 "t14_standardSMD:C2012m" V 3650 4200 30  0001 C CNN
@@
 AR Path="/5F69D945/5F69C099" Ref="C314"  Part="1"
 AR Path="/5F69D9BA/5F69C099" Ref="C414"  Part="1"
-F 0 "C314" V 6800 4350 40  0000 L CNN
+F 0 "C414" V 6800 4350 40  0000 L CNN
 F 1 "10u/25V" V 6900 4300 40  0000 L CNN
 F 2 "t14_standardSMD:C2012m" V 7000 4200 30  0001 C CNN
@@
 AR Path="/5F69D945/5F69C4C2" Ref="C315"  Part="1"
 AR Path="/5F69D9BA/5F69C4C2" Ref="C415"  Part="1"
-F 0 "C315" V 7000 4350 40  0000 L CNN
+F 0 "C415" V 7000 4350 40  0000 L CNN
 F 1 "10u/25V" V 7100 4300 40  0000 L CNN
 F 2 "t14_standardSMD:C2012m" V 7200 4200 30  0001 C CNN
@@
 AR Path="/5F69D945/5F69C649" Ref="C316"  Part="1"
 AR Path="/5F69D9BA/5F69C649" Ref="C416"  Part="1"
-F 0 "C316" V 7200 4350 40  0000 L CNN
+F 0 "C416" V 7200 4350 40  0000 L CNN
 F 1 "10u/25V" V 7300 4300 40  0000 L CNN
 F 2 "t14_standardSMD:C2012m" V 7400 4200 30  0001 C CNN
@@
 AR Path="/5F69D945/5F69C7C9" Ref="C317"  Part="1"
 AR Path="/5F69D9BA/5F69C7C9" Ref="C417"  Part="1"
-F 0 "C317" V 7400 4350 40  0000 L CNN
+F 0 "C417" V 7400 4350 40  0000 L CNN
 F 1 "10u/25V" V 7500 4300 40  0000 L CNN
 F 2 "t14_standardSMD:C2012m" V 7600 4200 30  0001 C CNN
@@
 AR Path="/5F69D945/5F69C9A2" Ref="C318"  Part="1"
 AR Path="/5F69D9BA/5F69C9A2" Ref="C418"  Part="1"
-F 0 "C318" V 7600 4350 40  0000 L CNN
+F 0 "C418" V 7600 4350 40  0000 L CNN
 F 1 "10u/25V" V 7700 4300 40  0000 L CNN
 F 2 "t14_standardSMD:C2012m" V 7800 4200 30  0001 C CNN
@@
 AR Path="/5F69D945/5F69CED4" Ref="C309"  Part="1"
 AR Path="/5F69D9BA/5F69CED4" Ref="C409"  Part="1"
-F 0 "C309" V 3950 4350 40  0000 L CNN
+F 0 "C409" V 3950 4350 40  0000 L CNN
 F 1 "100n/25V" V 4050 4300 40  0000 L CNN
 F 2 "t14_standardSMD:C1608m" V 4150 4200 30  0001 C CNN
@@
 AR Path="/5F69D945/5F69D10B" Ref="C310"  Part="1"
 AR Path="/5F69D9BA/5F69D10B" Ref="C410"  Part="1"
-F 0 "C310" V 4150 4350 40  0000 L CNN
+F 0 "C410" V 4150 4350 40  0000 L CNN
 F 1 "100n/25V" V 4250 4300 40  0000 L CNN
 F 2 "t14_standardSMD:C1608m" V 4350 4200 30  0001 C CNN
@@
 AR Path="/5F69D945/5F69D3A3" Ref="C311"  Part="1"
 AR Path="/5F69D9BA/5F69D3A3" Ref="C411"  Part="1"
-F 0 "C311" V 4350 4350 40  0000 L CNN
+F 0 "C411" V 4350 4350 40  0000 L CNN
 F 1 "100n/25V" V 4450 4300 40  0000 L CNN
 F 2 "t14_standardSMD:C1608m" V 4550 4200 30  0001 C CNN
